File: low_cost_bldc-power.kicad_sch (KiCad schematic)
At the start: 0 parts

Commit message: Top-only inverter layout
Other:
- title: (none) -> FreeWheel
Changed lines of the file:
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@@
 	(generator_version "8.0")
 	(paper "A4")
+	(title_block
+		(title "FreeWheel")
+		(rev "001")
+	)
 )
