File: Phase.kicad_sch (KiCad schematic)
At the start: 22 parts, among them Q1 HSCB3014, Q2 HSCB3014, U3 U2115C, U4 COS8051

Commit message: Organizing
Other:
- note added: "Fix gain w/ resistor"
- note added: "This resistor is gonna pop"
Changed lines of the file:
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@@
+		)
+	)
+	(text "This resistor is gonna pop"
+		(exclude_from_sim no)
+		(at 256.286 175.006 0)
+		(effects
+			(font
+				(size 1.27 1.27)
+			)
 		)
 	)
@@
 		(effects
 			(font
+				(size 1.27 1.27)
+			)
+		)
+	)
+	(text "Fix gain w/ resistor"
+		(exclude_from_sim no)
+		(at 205.74 177.546 0)
+		(effects
+			(font
